Commit message: updated

File: src/dogbot_description/dogbot/urdf/dogbot.urdf.xacro (robot description, xacro)
@@ -11,7 +11,8 @@
     <xacro:property name="wheel_len" value="0.02" />
     <xacro:property name="wheel_radius" value="0.015" />
-    <xacro:property name="z_offset" value="-${base_height/2}" /> <!-- Space btw top of beam and the each joint -->
+    <xacro:property name="z_offset" value="-${base_height/2}" /> <!-- Space btw top of beam and the
+    each joint -->
     <!-- Base Link -->
-    <link name="${prefix}base_link">
+    <link name="base_link">
       <collision>
         <origin xyz="0 0 0" rpy="0 0 0" />
@@ -27,18 +28,9 @@
         <material name="orange" />
       </visual>
-      <inertial>
-        <origin xyz="0 0 0" rpy="0 0 0" />
-        <mass value="${base_mass}" />
-        <inertia
-          ixx="${base_mass / 12.0 * (base_length*base_length + base_height*base_height)}" ixy="0.0"
-          ixz="0.0"
-          iyy="${base_mass / 12.0 * (base_height*base_height + base_width*base_width)}" iyz="0.0"
-          izz="${base_mass / 12.0 * (base_width*base_width + base_length*base_length)}" />
-      </inertial>
     </link>
     <!-- left front wheel joint -->
-    <joint name="${prefix}lf_wheel_joint" type="continuous">
-      <parent link="${prefix}base_link" />
-      <child link="${prefix}lf_wheel" />
+    <joint name="lf_wheel_joint" type="continuous">
+      <parent link="base_link" />
+      <child link="lf_wheel" />
       <origin xyz="0.03 -${base_width/2} ${z_offset}" rpy="0 0 0" />
       <axis xyz="0 1 0" />
@@ -47,5 +39,5 @@
     </joint>
     <!-- left front wheel Link -->
-    <link name="${prefix}lf_wheel">
+    <link name="lf_wheel">
       <collision>
         <origin xyz="0 0 0" rpy="${PI/2} 0 0" />
@@ -61,18 +53,9 @@
         <material name="black" />
       </visual>
-      <inertial>
-        <origin xyz="0 0 0" rpy="${PI/2} 0 0" />
-        <mass value="${wheel_mass}" />
-        <inertia
-          ixx="${wheel_mass / 12.0 * (3*wheel_radius*wheel_radius + wheel_len*wheel_len)}" ixy="0.0"
-          ixz="0.0"
-          iyy="${wheel_mass / 12.0 * (3*wheel_radius*wheel_radius + wheel_len*wheel_len)}" iyz="0.0"
-          izz="${wheel_mass / 2.0 * wheel_radius*wheel_radius}" />
-      </inertial>
     </link>
     <!-- right front wheel joint -->
-    <joint name="${prefix}rf_wheel_joint" type="continuous">
-      <parent link="${prefix}base_link" />
-      <child link="${prefix}rf_wheel" />
+    <joint name="rf_wheel_joint" type="continuous">
+      <parent link="base_link" />
+      <child link="rf_wheel" />
       <origin xyz="0.03 ${base_width/2} ${z_offset}" rpy="0 0 0" />
       <axis xyz="0 1 0" />
@@ -81,5 +64,5 @@
     </joint>
     <!-- right front wheel Link -->
-    <link name="${prefix}rf_wheel">
+    <link name="rf_wheel">
       <collision>
         <origin xyz="0 0 0" rpy="${PI/2} 0 0" />
@@ -95,18 +78,9 @@
         <material name="black" />
       </visual>
-      <inertial>
-        <origin xyz="0 0 0" rpy="${PI/2} 0 0" />
-        <mass value="${wheel_mass}" />
-        <inertia
-          ixx="${wheel_mass / 12.0 * (3*wheel_radius*wheel_radius + wheel_len*wheel_len)}" ixy="0.0"
-          ixz="0.0"
-          iyy="${wheel_mass / 12.0 * (3*wheel_radius*wheel_radius + wheel_len*wheel_len)}" iyz="0.0"
-          izz="${wheel_mass / 2.0 * wheel_radius*wheel_radius}" />
-      </inertial>
     </link>
     <!-- left back wheel joint -->
-    <joint name="${prefix}lb_wheel_joint" type="continuous">
-      <parent link="${prefix}base_link" />
-      <child link="${prefix}lb_wheel" />
+    <joint name="lb_wheel_joint" type="continuous">
+      <parent link="base_link" />
+      <child link="lb_wheel" />
       <origin xyz="-0.03 -${base_width/2} ${z_offset}" rpy="0 0 0" />
       <axis xyz="0 1 0" />
@@ -115,5 +89,5 @@
     </joint>
     <!-- left back wheel Link -->
-    <link name="${prefix}lb_wheel">
+    <link name="lb_wheel">
       <collision>
         <origin xyz="0 0 0" rpy="${PI/2} 0 0" />
@@ -129,18 +103,9 @@
         <material name="black" />
       </visual>
-      <inertial>
-        <origin xyz="0 0 0" rpy="${PI/2} 0 0" />
-        <mass value="${wheel_mass}" />
-        <inertia
-          ixx="${wheel_mass / 12.0 * (3*wheel_radius*wheel_radius + wheel_len*wheel_len)}" ixy="0.0"
-          ixz="0.0"
-          iyy="${wheel_mass / 12.0 * (3*wheel_radius*wheel_radius + wheel_len*wheel_len)}" iyz="0.0"
-          izz="${wheel_mass / 2.0 * wheel_radius*wheel_radius}" />
-      </inertial>
     </link>
     <!-- right back wheel joint -->
-    <joint name="${prefix}rb_wheel_joint" type="continuous">
-      <parent link="${prefix}base_link" />
-      <child link="${prefix}rb_wheel" />
+    <joint name="rb_wheel_joint" type="continuous">
+      <parent link="base_link" />
+      <child link="rb_wheel" />
       <origin xyz="-0.03 ${base_width/2} ${z_offset}" rpy="0 0 0" />
       <axis xyz="0 1 0" />
@@ -149,5 +114,5 @@
     </joint>
     <!-- right back wheel Link -->
-    <link name="${prefix}rb_wheel">
+    <link name="rb_wheel">
       <collision>
         <origin xyz="0 0 0" rpy="${PI/2} 0 0" />
@@ -163,13 +128,4 @@
         <material name="black" />
       </visual>
-      <inertial>
-        <origin xyz="0 0 0" rpy="${PI/2} 0 0" />
-        <mass value="${wheel_mass}" />
-        <inertia
-          ixx="${wheel_mass / 12.0 * (3*wheel_radius*wheel_radius + wheel_len*wheel_len)}" ixy="0.0"
-          ixz="0.0"
-          iyy="${wheel_mass / 12.0 * (3*wheel_radius*wheel_radius + wheel_len*wheel_len)}" iyz="0.0"
-          izz="${wheel_mass / 2.0 * wheel_radius*wheel_radius}" />
-      </inertial>
     </link>
   </xacro:macro>
