Commit message: added arm

File: dogbot_hardware/description/ros2_control/dogbot.ros2_control.xacro (robot description, xacro)
@@ -33,4 +33,16 @@
                 <state_interface name="position"/>
             </joint>
+            <joint name="${prefix}servo_gripper_joint">
+                <command_interface name="position"/>
+                <state_interface name="position"/>
+            </joint>
+            <joint name="${prefix}servo_shoulder_joint">
+                <command_interface name="position"/>
+                <state_interface name="position"/>
+            </joint>
+            <joint name="${prefix}servo_forearm_joint">
+                <command_interface name="position"/>
+                <state_interface name="position"/>
+            </joint>
         </ros2_control>
     </xacro:macro>

Commit message: dev

File: dogbot_hardware/description/ros2_control/dogbot.ros2_control.xacro (robot description, xacro)
@@ -33,5 +33,5 @@
                 <state_interface name="position"/>
             </joint>
-            <joint name="${prefix}servo_gripper_joint">
+            <!-- <joint name="${prefix}servo_gripper_joint">
                 <command_interface name="position"/>
                 <state_interface name="position"/>
@@ -44,5 +44,5 @@
                 <command_interface name="position"/>
                 <state_interface name="position"/>
-            </joint>
+            </joint> -->
         </ros2_control>
     </xacro:macro>
