Commit message: updated

File: dogbot_description/dogbot/urdf/dogbot.urdf.xacro (robot description, xacro)
@@ -1,132 +1,126 @@
 <?xml version="1.0"?>
 <robot xmlns:xacro="http://www.ros.org/wiki/xacro">
-  <xacro:macro name="dogbot" params="prefix">
-    <!-- Constants for robot dimensions -->
-    <xacro:property name="PI" value="3.1415926535897931" />
-    <xacro:property name="base_mass" value="0.3" /> <!-- arbitrary value for base mass -->
-    <xacro:property name="base_width" value="0.1" />
-    <xacro:property name="base_length" value="0.1" />
-    <xacro:property name="base_height" value="0.05" />
-    <xacro:property name="wheel_mass" value="0.3" /> <!-- arbitrary value for wheel mass -->
-    <xacro:property name="wheel_len" value="0.02" />
-    <xacro:property name="wheel_radius" value="0.015" />
-    <xacro:property name="z_offset" value="-${base_height/2}" /> <!-- Space btw top of beam and the
-    each joint -->
-    <!-- Base Link -->
-    <link name="base_link">
-      <collision>
-        <origin xyz="0 0 0" rpy="0 0 0" />
-        <geometry>
-          <box size="${base_width} ${base_length} ${base_height}" />
-        </geometry>
-      </collision>
-      <visual>
-        <origin xyz="0 0 ${base_height/2}" rpy="0 0 0" />
-        <geometry>
-          <box size="${base_width} ${base_length} ${base_height}" />
-        </geometry>
-        <material name="orange" />
-      </visual>
-    </link>
-    <!-- left front wheel joint -->
-    <joint name="lf_wheel_joint" type="continuous">
-      <parent link="base_link" />
-      <child link="lf_wheel" />
-      <origin xyz="0.03 -${base_width/2} ${z_offset}" rpy="0 0 0" />
-      <axis xyz="0 1 0" />
-      <dynamics damping="0.2" />
-      <limit effort="100" velocity="1.0" />
-    </joint>
-    <!-- left front wheel Link -->
-    <link name="lf_wheel">
-      <collision>
-        <origin xyz="0 0 0" rpy="${PI/2} 0 0" />
-        <geometry>
-          <cylinder length="${wheel_len}" radius="${wheel_radius}" />
-        </geometry>
-      </collision>
-      <visual>
-        <origin xyz="0 0 0" rpy="${PI/2} 0 0" />
-        <geometry>
-          <cylinder length="${wheel_len}" radius="${wheel_radius}" />
-        </geometry>
-        <material name="black" />
-      </visual>
-    </link>
-    <!-- right front wheel joint -->
-    <joint name="rf_wheel_joint" type="continuous">
-      <parent link="base_link" />
-      <child link="rf_wheel" />
-      <origin xyz="0.03 ${base_width/2} ${z_offset}" rpy="0 0 0" />
-      <axis xyz="0 1 0" />
-      <dynamics damping="0.2" />
-      <limit effort="100" velocity="1.0" />
-    </joint>
-    <!-- right front wheel Link -->
-    <link name="rf_wheel">
-      <collision>
-        <origin xyz="0 0 0" rpy="${PI/2} 0 0" />
-        <geometry>
-          <cylinder length="${wheel_len}" radius="${wheel_radius}" />
-        </geometry>
-      </collision>
-      <visual>
-        <origin xyz="0 0 0" rpy="${PI/2} 0 0" />
-        <geometry>
-          <cylinder length="${wheel_len}" radius="${wheel_radius}" />
-        </geometry>
-        <material name="black" />
-      </visual>
-    </link>
-    <!-- left back wheel joint -->
-    <joint name="lb_wheel_joint" type="continuous">
-      <parent link="base_link" />
-      <child link="lb_wheel" />
-      <origin xyz="-0.03 -${base_width/2} ${z_offset}" rpy="0 0 0" />
-      <axis xyz="0 1 0" />
-      <dynamics damping="0.2" />
-      <limit effort="100" velocity="1.0" />
-    </joint>
-    <!-- left back wheel Link -->
-    <link name="lb_wheel">
-      <collision>
-        <origin xyz="0 0 0" rpy="${PI/2} 0 0" />
-        <geometry>
-          <cylinder length="${wheel_len}" radius="${wheel_radius}" />
-        </geometry>
-      </collision>
-      <visual>
-        <origin xyz="0 0 0" rpy="${PI/2} 0 0" />
-        <geometry>
-          <cylinder length="${wheel_len}" radius="${wheel_radius}" />
-        </geometry>
-        <material name="black" />
-      </visual>
-    </link>
-    <!-- right back wheel joint -->
-    <joint name="rb_wheel_joint" type="continuous">
-      <parent link="base_link" />
-      <child link="rb_wheel" />
-      <origin xyz="-0.03 ${base_width/2} ${z_offset}" rpy="0 0 0" />
-      <axis xyz="0 1 0" />
-      <dynamics damping="0.2" />
-      <limit effort="100" velocity="1.0" />
-    </joint>
-    <!-- right back wheel Link -->
-    <link name="rb_wheel">
-      <collision>
-        <origin xyz="0 0 0" rpy="${PI/2} 0 0" />
-        <geometry>
-          <cylinder length="${wheel_len}" radius="${wheel_radius}" />
-        </geometry>
-      </collision>
-      <visual>
-        <origin xyz="0 0 0" rpy="${PI/2} 0 0" />
-        <geometry>
-          <cylinder length="${wheel_len}" radius="${wheel_radius}" />
-        </geometry>
-        <material name="black" />
-      </visual>
-    </link>
-  </xacro:macro>
+    <xacro:macro name="dogbot" params="prefix">
+        <!-- Constants for robot dimensions -->
+        <xacro:property name="PI" value="3.1415926535897931"/>
+        <xacro:property name="base_mass" value="1.5"/> <!-- arbitrary value for base mass -->
+        <xacro:property name="base_width" value="0.25"/>
+        <xacro:property name="base_length" value="0.15"/>
+        <xacro:property name="base_height" value="0.03"/>
+        <xacro:property name="base_z_offset" value="0.06"/>
+        <xacro:property name="wheel_mass" value="0.05"/> <!-- arbitrary value for wheel mass -->
+        <xacro:property name="wheel_len" value="0.04"/>
+        <xacro:property name="wheel_radius" value="0.04"/>
+        <xacro:property name="wheel_x_alignment" value="0.0875"/>
+        <xacro:property name="wheel_y_alignment" value="0.125"/>
+        <xacro:property name="wheel_joint_z_offset" value="0.04"/> <!-- Space btw top of beam and each joint -->
+        <!-- Base Link -->
+        <link name="base_link">
+            <collision>
+                <origin xyz="0 0 0" rpy="0 0 0"/>
+                <geometry>
+                    <box size="${base_width} ${base_length} ${base_height}"/>
+                </geometry>
+            </collision>
+            <visual>
+                <origin xyz="0 0 ${base_z_offset}" rpy="0 0 0"/>
+                <geometry>
+                    <box size="${base_width} ${base_length} ${base_height}"/>
+                </geometry>
+                <material name="orange"/>
+            </visual>
+        </link>
+        <!-- left front wheel joint -->
+        <joint name="lf_wheel_joint" type="fixed">
+            <parent link="base_link"/>
+            <child link="lf_wheel"/>
+            <origin xyz="${wheel_x_alignment} ${wheel_y_alignment} ${wheel_joint_z_offset}" rpy="0 0 0"/>
+            <axis xyz="0 1 0"/>
+        </joint>
+        <!-- left front wheel Link -->
+        <link name="lf_wheel">
+            <collision>
+                <origin xyz="0 0 0" rpy="${PI/2} 0 0"/>
+                <geometry>
+                    <cylinder length="${wheel_len}" radius="${wheel_radius}"/>
+                </geometry>
+            </collision>
+            <visual>
+                <origin xyz="0 0 0" rpy="${PI/2} 0 0"/>
+                <geometry>
+                    <cylinder length="${wheel_len}" radius="${wheel_radius}"/>
+                </geometry>
+                <material name="black"/>
+            </visual>
+        </link>
+        <!-- right front wheel joint -->
+        <joint name="rf_wheel_joint" type="continuous">
+            <parent link="base_link"/>
+            <child link="rf_wheel"/>
+            <origin xyz="${wheel_x_alignment} -${wheel_y_alignment} ${wheel_joint_z_offset}" rpy="0 0 0"/>
+            <axis xyz="0 1 0"/>
+        </joint>
+        <!-- right front wheel Link -->
+        <link name="rf_wheel">
+            <collision>
+                <origin xyz="0 0 0" rpy="${PI/2} 0 0"/>
+                <geometry>
+                    <cylinder length="${wheel_len}" radius="${wheel_radius}"/>
+                </geometry>
+            </collision>
+            <visual>
+                <origin xyz="0 0 0" rpy="${PI/2} 0 0"/>
+                <geometry>
+                    <cylinder length="${wheel_len}" radius="${wheel_radius}"/>
+                </geometry>
+                <material name="black"/>
+            </visual>
+        </link>
+        <!-- left back wheel joint -->
+        <joint name="lb_wheel_joint" type="continuous">
+            <parent link="base_link"/>
+            <child link="lb_wheel"/>
+            <origin xyz="-${wheel_x_alignment} ${wheel_y_alignment} ${wheel_joint_z_offset}" rpy="0 0 0"/>
+            <axis xyz="0 1 0"/>
+        </joint>
+        <!-- left back wheel Link -->
+        <link name="lb_wheel">
+            <collision>
+                <origin xyz="0 0 0" rpy="${PI/2} 0 0"/>
+                <geometry>
+                    <cylinder length="${wheel_len}" radius="${wheel_radius}"/>
+                </geometry>
+            </collision>
+            <visual>
+                <origin xyz="0 0 0" rpy="${PI/2} 0 0"/>
+                <geometry>
+                    <cylinder length="${wheel_len}" radius="${wheel_radius}"/>
+                </geometry>
+                <material name="black"/>
+            </visual>
+        </link>
+        <!-- right back wheel joint -->
+        <joint name="rb_wheel_joint" type="continuous">
+            <parent link="base_link"/>
+            <child link="rb_wheel"/>
+            <origin xyz="-${wheel_x_alignment} -${wheel_y_alignment} ${wheel_joint_z_offset}" rpy="0 0 0"/>
+            <axis xyz="0 1 0"/>
+        </joint>
+        <!-- right back wheel Link -->
+        <link name="rb_wheel">
+            <collision>
+                <origin xyz="0 0 0" rpy="${PI/2} 0 0"/>
+                <geometry>
+                    <cylinder length="${wheel_len}" radius="${wheel_radius}"/>
+                </geometry>
+            </collision>
+            <visual>
+                <origin xyz="0 0 0" rpy="${PI/2} 0 0"/>
+                <geometry>
+                    <cylinder length="${wheel_len}" radius="${wheel_radius}"/>
+                </geometry>
+                <material name="black"/>
+            </visual>
+        </link>
+    </xacro:macro>
 </robot>

File: dogbot_hardware/description/ros2_control/dogbot.ros2_control.xacro (robot description, xacro)
@@ -1,45 +1,34 @@
 <?xml version="1.0"?>
 <robot xmlns:xacro="http://www.ros.org/wiki/xacro">
-  <xacro:macro name="dogbot_ros2_control" params="name prefix use_mock_hardware">
-    <ros2_control name="${name}" type="system">
-      <xacro:unless value="${use_mock_hardware}">
-        <hardware>
-          <plugin>dogbot_hardware/DogBotSystemHardware</plugin>
-          <param name="lf_wheel_name">lf_wheel_joint</param>
-          <param name="rf_wheel_name">rf_wheel_joint</param>
-          <param name="lb_wheel_name">lb_wheel_joint</param>
-          <param name="rb_wheel_name">rb_wheel_joint</param>
-          <param name="device">/dev/arduino</param>
-          <param name="baud_rate">115200</param>
-          <param name="timeout_ms">100</param>
-        </hardware>
-      </xacro:unless>
-      <xacro:if value="${use_mock_hardware}">
-        <hardware>
-          <plugin>mock_components/GenericSystem</plugin>
-          <param name="calculate_dynamics">true</param>
-        </hardware>
-      </xacro:if>
-      <joint name="${prefix}lf_wheel_joint">
-        <command_interface name="velocity" />
-        <state_interface name="position" />
-        <state_interface name="velocity" />
-      </joint>
-      <joint name="${prefix}rf_wheel_joint">
-        <command_interface name="velocity" />
-        <state_interface name="position" />
-        <state_interface name="velocity" />
-      </joint>
-      <joint name="${prefix}lb_wheel_joint">
-        <command_interface name="velocity" />
-        <state_interface name="position" />
-        <state_interface name="velocity" />
-      </joint>
-      <joint name="${prefix}rb_wheel_joint">
-        <command_interface name="velocity" />
-        <state_interface name="position" />
-        <state_interface name="velocity" />
-      </joint>
-    </ros2_control>
-  </xacro:macro>
+    <xacro:macro name="dogbot_ros2_control" params="name prefix">
+        <ros2_control name="${name}" type="system">
+            <hardware>
+                <plugin>dogbot_hardware/DogBotSystemHardware</plugin>
+                <param name="lf_wheel_name">lf_wheel_joint</param>
+                <param name="rf_wheel_name">rf_wheel_joint</param>
+                <param name="lb_wheel_name">lb_wheel_joint</param>
+                <param name="rb_wheel_name">rb_wheel_joint</param>
+                <param name="device">/dev/arduino</param>
+                <param name="baud_rate">115200</param>
+                <param name="timeout_ms">1000</param>
+                <param name="enc_counts_per_rev">1320</param>
+            </hardware>s
+            <joint name="${prefix}lf_wheel_joint">
+                <command_interface name="velocity"/>
+                <state_interface name="position"/>
+            </joint>
+            <joint name="${prefix}rf_wheel_joint">
+                <command_interface name="velocity"/>
+                <state_interface name="position"/>
+            </joint>
+            <joint name="${prefix}lb_wheel_joint">
+                <command_interface name="velocity"/>
+                <state_interface name="position"/>
+            </joint>
+            <joint name="${prefix}rb_wheel_joint">
+                <command_interface name="velocity"/>
+                <state_interface name="position"/>
+            </joint>
+        </ros2_control>
+    </xacro:macro>
 </robot>

File: dogbot_hardware/description/urdf/dogbot.urdf.xacro (robot description, xacro)
@@ -3,5 +3,4 @@
 <robot xmlns:xacro="http://www.ros.org/wiki/xacro" name="dogbot_base">
   <xacro:arg name="prefix" default="" />
-  <xacro:arg name="use_mock_hardware" default="false" />
   <xacro:include filename="$(find dogbot_description)/dogbot/urdf/dogbot.urdf.xacro" />
   <!-- Import Rviz colors -->
@@ -11,4 +10,4 @@
   <xacro:dogbot prefix="$(arg prefix)" />
   <xacro:dogbot_ros2_control
-    name="DogBot" prefix="$(arg prefix)" use_mock_hardware="$(arg use_mock_hardware)"/>
+    name="DogBot" prefix="$(arg prefix)"/>
 </robot>

Commit message: Added arm support

File: dogbot_description/dogbot/urdf/dogbot.urdf.xacro (robot description, xacro)
@@ -123,4 +123,55 @@
             </visual>
         </link>
+        <!-- arm forearm joint -->
+        <joint name="servo_forearm_joint" type="continuous">
+            <parent link="base_link"/>
+            <child link="servo_forearm"/>
+            <origin xyz="0 0 0" rpy="0 0 0"/>
+            <axis xyz="0 1 0"/>
+        </joint>
+        <!-- arm forearm Link -->
+        <link name="servo_forearm">
+            <visual>
+                <origin xyz="0 0 0" rpy="0 0 0"/>
+                <geometry>
+                    <box size="0.1 0.1 0.1"/>
+                </geometry>
+                <material name="green"/>
+            </visual>
+        </link>
+        <!-- arm shoulder joint -->
+        <joint name="servo_shoulder_joint" type="continuous">
+            <parent link="servo_forearm"/>
+            <child link="servo_shoulder"/>
+            <origin xyz="0 0 0" rpy="0 0 0"/>
+            <axis xyz="0 1 0"/>
+        </joint>
+        <!-- arm shoulder Link -->
+        <link name="servo_shoulder">
+            <visual>
+                <origin xyz="0 0 0" rpy="0 0 0"/>
+                <geometry>
+                    <box size="0.1 0.1 0.1"/>
+                </geometry>
+                <material name="green"/>
+            </visual>
+        </link>
+        <!-- arm gripper joint -->
+        <joint name="servo_gripper_joint" type="continuous">
+            <parent link="servo_shoulder"/>
+            <child link="servo_gripper"/>
+            <origin xyz="0 0 0" rpy="0 0 0"/>
+            <axis xyz="0 1 0"/>
+        </joint>
+        <!-- arm gripper Link -->
+        <link name="servo_gripper">
+            <visual>
+                <origin xyz="0 0 0" rpy="0 0 0"/>
+                <geometry>
+                    <box size="0.1 0.1 0.1"/>
+                </geometry>
+                <material name="green"/>
+            </visual>
+        </link>
     </xacro:macro>
 </robot>

File: dogbot_hardware/description/ros2_control/dogbot.ros2_control.xacro (robot description, xacro)
@@ -9,4 +9,7 @@
                 <param name="lb_wheel_name">lb_wheel_joint</param>
                 <param name="rb_wheel_name">rb_wheel_joint</param>
+                <param name="servo_gripper_name">servo_gripper_joint</param>
+                <param name="servo_shoulder_name">servo_shoulder_joint</param>
+                <param name="servo_forearm_name">servo_forearm_joint</param>
                 <param name="device">/dev/arduino</param>
                 <param name="baud_rate">115200</param>
