Commit message: added slam support

File: dogbot_description/dogbot/urdf/dogbot.urdf.xacro (robot description, xacro)
@@ -3,173 +3,218 @@
     <xacro:macro name="dogbot" params="prefix">
         <!-- Constants for robot dimensions -->
-        <xacro:property name="PI" value="3.1415926535897931"/>
-        <xacro:property name="base_mass" value="1.5"/> <!-- arbitrary value for base mass -->
-        <xacro:property name="base_width" value="0.25"/>
-        <xacro:property name="base_length" value="0.15"/>
-        <xacro:property name="base_height" value="0.03"/>
-        <xacro:property name="base_z_offset" value="0.06"/>
-        <xacro:property name="wheel_mass" value="0.05"/> <!-- arbitrary value for wheel mass -->
-        <xacro:property name="wheel_len" value="0.04"/>
-        <xacro:property name="wheel_radius" value="0.04"/>
-        <xacro:property name="wheel_x_alignment" value="0.0875"/>
-        <xacro:property name="wheel_y_alignment" value="0.125"/>
-        <xacro:property name="wheel_joint_z_offset" value="0.04"/> <!-- Space btw top of beam and each joint -->
+        <xacro:property name="PI" value="3.1415926535897931" />
+        <xacro:property name="base_mass" value="1.5" /> <!-- arbitrary value for base mass -->
+        <xacro:property name="base_width" value="0.25" />
+        <xacro:property name="base_length" value="0.15" />
+        <xacro:property name="base_height" value="0.03" />
+        <xacro:property name="base_z_offset" value="0.06" />
+        <xacro:property name="wheel_mass" value="0.05" /> <!-- arbitrary value for wheel mass -->
+        <xacro:property name="wheel_len" value="0.04" />
+        <xacro:property name="wheel_radius" value="0.04" />
+        <xacro:property name="wheel_x_alignment" value="0.0875" />
+        <xacro:property name="wheel_y_alignment" value="0.125" />
+        <xacro:property name="wheel_joint_z_offset" value="0.04" /> <!-- Space btw top of beam and
+        each joint -->
+        <!-- Robot Footprint -->
+        <link name="base_footprint" />
+        <joint name="base_joint" type="fixed">
+            <parent link="base_footprint" />
+            <child link="base_link" />
+            <origin xyz="0 0 0" rpy="0 0 0" />
+        </joint>
         <!-- Base Link -->
         <link name="base_link">
             <collision>
-                <origin xyz="0 0 0" rpy="0 0 0"/>
-                <geometry>
-                    <box size="${base_width} ${base_length} ${base_height}"/>
-                </geometry>
-            </collision>
-            <visual>
-                <origin xyz="0 0 ${base_z_offset}" rpy="0 0 0"/>
-                <geometry>
-                    <box size="${base_width} ${base_length} ${base_height}"/>
-                </geometry>
-                <material name="orange"/>
-            </visual>
-        </link>
+                <origin xyz="0 0 0" rpy="0 0 0" />
+                <geometry>
+                    <box size="${base_width} ${base_length} ${base_height}" />
+                </geometry>
+            </collision>
+            <visual>
+                <origin xyz="0 0 ${base_z_offset}" rpy="0 0 0" />
+                <geometry>
+                    <box size="${base_width} ${base_length} ${base_height}" />
+                </geometry>
+                <material name="orange" />
+            </visual>
+        </link>
+        <!-- laser link -->
+        <link name="laser_frame">
+            <visual>
+                <origin xyz="0 0 0" rpy="0 0 0" />
+                <geometry>
+                    <cylinder length="0.02" radius="0.02" />
+                </geometry>
+                <material name="black">
+                    <color rgba="0.0 0.0 0.0 0.5" />
+                </material>
+            </visual>
+        </link>
+        <!-- laser joint -->
+        <joint name="laser_joint" type="fixed">
+            <parent link="base_link" />
+            <child link="laser_frame" />
+            <origin xyz="0 0 0.075" />
+        </joint>
+        <!-- imu link -->
+        <link name="imu_link">
+            <visual>
+                <origin xyz="0 0 0.0" rpy="0 0 0" />
+                <geometry>
+                    <box size="0.02 0.02 0.02" />
+                </geometry>
+            </visual>
+        </link>
+        <!-- imu joint -->
+        <joint name="imu_joint" type="fixed">
+            <parent link="base_link" />
+            <child link="imu_link" />
+            <origin xyz="0 0 0.02" />
+        </joint>
         <!-- left front wheel joint -->
         <joint name="lf_wheel_joint" type="fixed">
-            <parent link="base_link"/>
-            <child link="lf_wheel"/>
-            <origin xyz="${wheel_x_alignment} ${wheel_y_alignment} ${wheel_joint_z_offset}" rpy="0 0 0"/>
-            <axis xyz="0 1 0"/>
+            <parent link="base_link" />
+            <child link="lf_wheel" />
+            <origin xyz="${wheel_x_alignment} ${wheel_y_alignment} ${wheel_joint_z_offset}"
+                rpy="0 0 0" />
+            <axis xyz="0 1 0" />
         </joint>
         <!-- left front wheel Link -->
         <link name="lf_wheel">
             <collision>
-                <origin xyz="0 0 0" rpy="${PI/2} 0 0"/>
-                <geometry>
-                    <cylinder length="${wheel_len}" radius="${wheel_radius}"/>
-                </geometry>
-            </collision>
-            <visual>
-                <origin xyz="0 0 0" rpy="${PI/2} 0 0"/>
-                <geometry>
-                    <cylinder length="${wheel_len}" radius="${wheel_radius}"/>
-                </geometry>
-                <material name="black"/>
+                <origin xyz="0 0 0" rpy="${PI/2} 0 0" />
+                <geometry>
+                    <cylinder length="${wheel_len}" radius="${wheel_radius}" />
+                </geometry>
+            </collision>
+            <visual>
+                <origin xyz="0 0 0" rpy="${PI/2} 0 0" />
+                <geometry>
+                    <cylinder length="${wheel_len}" radius="${wheel_radius}" />
+                </geometry>
+                <material name="black" />
             </visual>
         </link>
         <!-- right front wheel joint -->
         <joint name="rf_wheel_joint" type="continuous">
-            <parent link="base_link"/>
-            <child link="rf_wheel"/>
-            <origin xyz="${wheel_x_alignment} -${wheel_y_alignment} ${wheel_joint_z_offset}" rpy="0 0 0"/>
-            <axis xyz="0 1 0"/>
+            <parent link="base_link" />
+            <child link="rf_wheel" />
+            <origin xyz="${wheel_x_alignment} -${wheel_y_alignment} ${wheel_joint_z_offset}"
+                rpy="0 0 0" />
+            <axis xyz="0 1 0" />
         </joint>
         <!-- right front wheel Link -->
         <link name="rf_wheel">
             <collision>
-                <origin xyz="0 0 0" rpy="${PI/2} 0 0"/>
-                <geometry>
-                    <cylinder length="${wheel_len}" radius="${wheel_radius}"/>
-                </geometry>
-            </collision>
-            <visual>
-                <origin xyz="0 0 0" rpy="${PI/2} 0 0"/>
-                <geometry>
-                    <cylinder length="${wheel_len}" radius="${wheel_radius}"/>
-                </geometry>
-                <material name="black"/>
+                <origin xyz="0 0 0" rpy="${PI/2} 0 0" />
+                <geometry>
+                    <cylinder length="${wheel_len}" radius="${wheel_radius}" />
+                </geometry>
+            </collision>
+            <visual>
+                <origin xyz="0 0 0" rpy="${PI/2} 0 0" />
+                <geometry>
+                    <cylinder length="${wheel_len}" radius="${wheel_radius}" />
+                </geometry>
+                <material name="black" />
             </visual>
         </link>
         <!-- left back wheel joint -->
         <joint name="lb_wheel_joint" type="continuous">
-            <parent link="base_link"/>
-            <child link="lb_wheel"/>
-            <origin xyz="-${wheel_x_alignment} ${wheel_y_alignment} ${wheel_joint_z_offset}" rpy="0 0 0"/>
-            <axis xyz="0 1 0"/>
+            <parent link="base_link" />
+            <child link="lb_wheel" />
+            <origin xyz="-${wheel_x_alignment} ${wheel_y_alignment} ${wheel_joint_z_offset}"
+                rpy="0 0 0" />
+            <axis xyz="0 1 0" />
         </joint>
         <!-- left back wheel Link -->
         <link name="lb_wheel">
             <collision>
-                <origin xyz="0 0 0" rpy="${PI/2} 0 0"/>
-                <geometry>
-                    <cylinder length="${wheel_len}" radius="${wheel_radius}"/>
-                </geometry>
-            </collision>
-            <visual>
-                <origin xyz="0 0 0" rpy="${PI/2} 0 0"/>
-                <geometry>
-                    <cylinder length="${wheel_len}" radius="${wheel_radius}"/>
-                </geometry>
-                <material name="black"/>
+                <origin xyz="0 0 0" rpy="${PI/2} 0 0" />
+                <geometry>
+                    <cylinder length="${wheel_len}" radius="${wheel_radius}" />
+                </geometry>
+            </collision>
+            <visual>
+                <origin xyz="0 0 0" rpy="${PI/2} 0 0" />
+                <geometry>
+                    <cylinder length="${wheel_len}" radius="${wheel_radius}" />
+                </geometry>
+                <material name="black" />
             </visual>
         </link>
         <!-- right back wheel joint -->
         <joint name="rb_wheel_joint" type="continuous">
-            <parent link="base_link"/>
-            <child link="rb_wheel"/>
-            <origin xyz="-${wheel_x_alignment} -${wheel_y_alignment} ${wheel_joint_z_offset}" rpy="0 0 0"/>
-            <axis xyz="0 1 0"/>
+            <parent link="base_link" />
+            <child link="rb_wheel" />
+            <origin xyz="-${wheel_x_alignment} -${wheel_y_alignment} ${wheel_joint_z_offset}"
+                rpy="0 0 0" />
+            <axis xyz="0 1 0" />
         </joint>
         <!-- right back wheel Link -->
         <link name="rb_wheel">
             <collision>
-                <origin xyz="0 0 0" rpy="${PI/2} 0 0"/>
-                <geometry>
-                    <cylinder length="${wheel_len}" radius="${wheel_radius}"/>
-                </geometry>
-            </collision>
-            <visual>
-                <origin xyz="0 0 0" rpy="${PI/2} 0 0"/>
-                <geometry>
-                    <cylinder length="${wheel_len}" radius="${wheel_radius}"/>
-                </geometry>
-                <material name="black"/>
+                <origin xyz="0 0 0" rpy="${PI/2} 0 0" />
+                <geometry>
+                    <cylinder length="${wheel_len}" radius="${wheel_radius}" />
+                </geometry>
+            </collision>
+            <visual>
+                <origin xyz="0 0 0" rpy="${PI/2} 0 0" />
+                <geometry>
+                    <cylinder length="${wheel_len}" radius="${wheel_radius}" />
+                </geometry>
+                <material name="black" />
             </visual>
         </link>
         <!-- arm forearm joint -->
         <joint name="servo_forearm_joint" type="continuous">
-            <parent link="base_link"/>
-            <child link="servo_forearm"/>
-            <origin xyz="0 0 0" rpy="0 0 0"/>
-            <axis xyz="0 1 0"/>
+            <parent link="base_link" />
+            <child link="servo_forearm" />
+            <origin xyz="0 0 0" rpy="0 0 0" />
+            <axis xyz="0 1 0" />
         </joint>
         <!-- arm forearm Link -->
         <link name="servo_forearm">
             <visual>
-                <origin xyz="0 0 0" rpy="0 0 0"/>
-                <geometry>
-                    <box size="0.1 0.1 0.1"/>
-                </geometry>
-                <material name="green"/>
+                <origin xyz="0 0 0" rpy="0 0 0" />
+                <geometry>
+                    <box size="0.1 0.1 0.1" />
+                </geometry>
+                <material name="green" />
             </visual>
         </link>
         <!-- arm shoulder joint -->
         <joint name="servo_shoulder_joint" type="continuous">
-            <parent link="servo_forearm"/>
-            <child link="servo_shoulder"/>
-            <origin xyz="0 0 0" rpy="0 0 0"/>
-            <axis xyz="0 1 0"/>
+            <parent link="servo_forearm" />
+            <child link="servo_shoulder" />
+            <origin xyz="0 0 0" rpy="0 0 0" />
+            <axis xyz="0 1 0" />
         </joint>
         <!-- arm shoulder Link -->
         <link name="servo_shoulder">
             <visual>
-                <origin xyz="0 0 0" rpy="0 0 0"/>
-                <geometry>
-                    <box size="0.1 0.1 0.1"/>
-                </geometry>
-                <material name="green"/>
+                <origin xyz="0 0 0" rpy="0 0 0" />
+                <geometry>
+                    <box size="0.1 0.1 0.1" />
+                </geometry>
+                <material name="green" />
             </visual>
         </link>
         <!-- arm gripper joint -->
         <joint name="servo_gripper_joint" type="continuous">
-            <parent link="servo_shoulder"/>
-            <child link="servo_gripper"/>
-            <origin xyz="0 0 0" rpy="0 0 0"/>
-            <axis xyz="0 1 0"/>
+            <parent link="servo_shoulder" />
+            <child link="servo_gripper" />
+            <origin xyz="0 0 0" rpy="0 0 0" />
+            <axis xyz="0 1 0" />
         </joint>
         <!-- arm gripper Link -->
         <link name="servo_gripper">
             <visual>
-                <origin xyz="0 0 0" rpy="0 0 0"/>
-                <geometry>
-                    <box size="0.1 0.1 0.1"/>
-                </geometry>
-                <material name="green"/>
+                <origin xyz="0 0 0" rpy="0 0 0" />
+                <geometry>
+                    <box size="0.1 0.1 0.1" />
+                </geometry>
+                <material name="green" />
             </visual>
         </link>

Commit message: updated controllers

File: dogbot_description/dogbot/urdf/dogbot.urdf.xacro (robot description, xacro)
@@ -16,11 +16,4 @@
         <xacro:property name="wheel_joint_z_offset" value="0.04" /> <!-- Space btw top of beam and
         each joint -->
-        <!-- Robot Footprint -->
-        <link name="base_footprint" />
-        <joint name="base_joint" type="fixed">
-            <parent link="base_footprint" />
-            <child link="base_link" />
-            <origin xyz="0 0 0" rpy="0 0 0" />
-        </joint>
         <!-- Base Link -->
         <link name="base_link">
@@ -168,7 +161,58 @@
             </visual>
         </link>
+        <!-- servo pan joint -->
+        <joint name="servo_pan_joint" type="continuous">
+            <parent link="base_link" />
+            <child link="servo_pan" />
+            <origin xyz="0 0 0" rpy="0 0 0" />
+            <axis xyz="0 1 0" />
+        </joint>
+        <!-- servo pan Link -->
+        <link name="servo_pan">
+            <visual>
+                <origin xyz="0 0 0" rpy="0 0 0" />
+                <geometry>
+                    <box size="0.05 0.05 0.05" />
+                </geometry>
+                <material name="green" />
+            </visual>
+        </link>
+        <!-- servo tilt joint -->
+        <joint name="servo_tilt_joint" type="continuous">
+            <parent link="servo_pan" />
+            <child link="servo_tilt" />
+            <origin xyz="0 0 0" rpy="0 0 0" />
+            <axis xyz="0 1 0" />
+        </joint>
+        <!-- servo tilt Link -->
+        <link name="servo_tilt">
+            <visual>
+                <origin xyz="0 0 0" rpy="0 0 0" />
+                <geometry>
+                    <box size="0.05 0.05 0.05" />
+                </geometry>
+                <material name="green" />
+            </visual>
+        </link>
+        <!-- servo shoulder joint -->
+        <joint name="servo_shoulder_joint" type="continuous">
+            <parent link="base_link" />
+            <child link="servo_shoulder" />
+            <origin xyz="0 0 0" rpy="0 0 0" />
+            <axis xyz="0 1 0" />
+        </joint>
+        <!-- servo shoulder Link -->
+        <link name="servo_shoulder">
+            <visual>
+                <origin xyz="0 0 0" rpy="0 0 0" />
+                <geometry>
+                    <box size="0.05 0.05 0.05" />
+                </geometry>
+                <material name="green" />
+            </visual>
+        </link>
         <!-- servo forearm joint -->
         <joint name="servo_forearm_joint" type="continuous">
-            <parent link="base_link" />
+            <parent link="servo_shoulder" />
             <child link="servo_forearm" />
             <origin xyz="0 0 0" rpy="0 0 0" />
@@ -180,22 +224,5 @@
                 <origin xyz="0 0 0" rpy="0 0 0" />
                 <geometry>
-                    <box size="0.1 0.1 0.1" />
-                </geometry>
-                <material name="green" />
-            </visual>
-        </link>
-        <!-- servo shoulder joint -->
-        <joint name="servo_shoulder_joint" type="continuous">
-            <parent link="servo_forearm" />
-            <child link="servo_shoulder" />
-            <origin xyz="0 0 0" rpy="0 0 0" />
-            <axis xyz="0 1 0" />
-        </joint>
-        <!-- servo shoulder Link -->
-        <link name="servo_shoulder">
-            <visual>
-                <origin xyz="0 0 0" rpy="0 0 0" />
-                <geometry>
-                    <box size="0.1 0.1 0.1" />
+                    <box size="0.05 0.05 0.05" />
                 </geometry>
                 <material name="green" />
@@ -204,5 +231,5 @@
         <!-- servo gripper joint -->
         <joint name="servo_gripper_joint" type="continuous">
-            <parent link="servo_shoulder" />
+            <parent link="servo_forearm" />
             <child link="servo_gripper" />
             <origin xyz="0 0 0" rpy="0 0 0" />
@@ -214,5 +241,5 @@
                 <origin xyz="0 0 0" rpy="0 0 0" />
                 <geometry>
-                    <box size="0.1 0.1 0.1" />
+                    <box size="0.05 0.05 0.05" />
                 </geometry>
                 <material name="green" />

File: dogbot_hardware/description/ros2_control/dogbot.ros2_control.xacro (robot description, xacro)
@@ -9,7 +9,9 @@
                 <param name="lb_wheel_name">lb_wheel_joint</param>
                 <param name="rb_wheel_name">rb_wheel_joint</param>
-                <param name="servo_gripper_name">servo_gripper_joint</param>
+                <param name="servo_pan_name">servo_pan_joint</param>
+                <param name="servo_tilt_name">servo_tilt_joint</param>
                 <param name="servo_shoulder_name">servo_shoulder_joint</param>
                 <param name="servo_forearm_name">servo_forearm_joint</param>
+                <param name="servo_gripper_name">servo_gripper_joint</param>
                 <param name="device">/dev/arduino</param>
                 <param name="baud_rate">115200</param>
@@ -18,31 +20,39 @@
             </hardware>
             <joint name="${prefix}lf_wheel_joint">
-                <command_interface name="velocity"/>
-                <state_interface name="position"/>
+                <command_interface name="velocity" />
+                <state_interface name="position" />
             </joint>
             <joint name="${prefix}rf_wheel_joint">
-                <command_interface name="velocity"/>
-                <state_interface name="position"/>
+                <command_interface name="velocity" />
+                <state_interface name="position" />
             </joint>
             <joint name="${prefix}lb_wheel_joint">
-                <command_interface name="velocity"/>
-                <state_interface name="position"/>
+                <command_interface name="velocity" />
+                <state_interface name="position" />
             </joint>
             <joint name="${prefix}rb_wheel_joint">
-                <command_interface name="velocity"/>
-                <state_interface name="position"/>
+                <command_interface name="velocity" />
+                <state_interface name="position" />
             </joint>
-            <!-- <joint name="${prefix}servo_gripper_joint">
-                <command_interface name="position"/>
-                <state_interface name="position"/>
+            <joint name="${prefix}servo_pan_joint">
+                <command_interface name="position" />
+                <state_interface name="position" />
+            </joint>
+            <joint name="${prefix}servo_tilt_joint">
+                <command_interface name="position" />
+                <state_interface name="position" />
             </joint>
             <joint name="${prefix}servo_shoulder_joint">
-                <command_interface name="position"/>
-                <state_interface name="position"/>
+                <command_interface name="position" />
+                <state_interface name="position" />
             </joint>
             <joint name="${prefix}servo_forearm_joint">
-                <command_interface name="position"/>
-                <state_interface name="position"/>
-            </joint> -->
+                <command_interface name="position" />
+                <state_interface name="position" />
+            </joint>
+            <joint name="${prefix}servo_gripper_joint">
+                <command_interface name="position" />
+                <state_interface name="position" />
+            </joint>
         </ros2_control>
     </xacro:macro>
