Commit message: removed servo pan, tilt, shoulder

File: dogbot_description/dogbot/urdf/dogbot.urdf.xacro (robot description, xacro)
@@ -161,58 +161,7 @@
             </visual>
         </link>
-        <!-- servo pan joint -->
-        <joint name="servo_pan_joint" type="continuous">
-            <parent link="base_link" />
-            <child link="servo_pan" />
-            <origin xyz="0 0 0" rpy="0 0 0" />
-            <axis xyz="0 1 0" />
-        </joint>
-        <!-- servo pan Link -->
-        <link name="servo_pan">
-            <visual>
-                <origin xyz="0 0 0" rpy="0 0 0" />
-                <geometry>
-                    <box size="0.05 0.05 0.05" />
-                </geometry>
-                <material name="green" />
-            </visual>
-        </link>
-        <!-- servo tilt joint -->
-        <joint name="servo_tilt_joint" type="continuous">
-            <parent link="servo_pan" />
-            <child link="servo_tilt" />
-            <origin xyz="0 0 0" rpy="0 0 0" />
-            <axis xyz="0 1 0" />
-        </joint>
-        <!-- servo tilt Link -->
-        <link name="servo_tilt">
-            <visual>
-                <origin xyz="0 0 0" rpy="0 0 0" />
-                <geometry>
-                    <box size="0.05 0.05 0.05" />
-                </geometry>
-                <material name="green" />
-            </visual>
-        </link>
-        <!-- servo shoulder joint -->
-        <joint name="servo_shoulder_joint" type="continuous">
-            <parent link="base_link" />
-            <child link="servo_shoulder" />
-            <origin xyz="0 0 0" rpy="0 0 0" />
-            <axis xyz="0 1 0" />
-        </joint>
-        <!-- servo shoulder Link -->
-        <link name="servo_shoulder">
-            <visual>
-                <origin xyz="0 0 0" rpy="0 0 0" />
-                <geometry>
-                    <box size="0.05 0.05 0.05" />
-                </geometry>
-                <material name="green" />
-            </visual>
-        </link>
         <!-- servo forearm joint -->
         <joint name="servo_forearm_joint" type="continuous">
-            <parent link="servo_shoulder" />
+            <parent link="base_link" />
             <child link="servo_forearm" />
             <origin xyz="0 0 0" rpy="0 0 0" />

File: dogbot_hardware/description/ros2_control/dogbot.ros2_control.xacro (robot description, xacro)
@@ -9,7 +9,4 @@
                 <param name="lb_wheel_name">lb_wheel_joint</param>
                 <param name="rb_wheel_name">rb_wheel_joint</param>
-                <param name="servo_pan_name">servo_pan_joint</param>
-                <param name="servo_tilt_name">servo_tilt_joint</param>
-                <param name="servo_shoulder_name">servo_shoulder_joint</param>
                 <param name="servo_forearm_name">servo_forearm_joint</param>
                 <param name="servo_gripper_name">servo_gripper_joint</param>
@@ -35,13 +32,4 @@
                 <state_interface name="position" />
             </joint>
-            <joint name="${prefix}servo_pan_joint">
-                <command_interface name="position" />
-            </joint>
-            <joint name="${prefix}servo_tilt_joint">
-                <command_interface name="position" />
-            </joint>
-            <joint name="${prefix}servo_shoulder_joint">
-                <command_interface name="position" />
-            </joint>
             <joint name="${prefix}servo_forearm_joint">
                 <command_interface name="position" />

Commit message: added sonars

File: dogbot_description/dogbot/urdf/dogbot.urdf.xacro (robot description, xacro)
@@ -195,4 +195,20 @@
             </visual>
         </link>
+        <!-- sonar joint -->
+        <joint name="sonar_joint" type="fixed">
+            <parent link="servo_gripper" />
+            <child link="sonar" />
+            <origin xyz="0 0 0" rpy="0 0 0" />
+        </joint>
+        <!-- sonar Link -->
+        <link name="sonar">
+            <visual>
+                <origin xyz="0 0 0" rpy="0 0 0" />
+                <geometry>
+                    <box size="0.01 0.01 0.01" />
+                </geometry>
+                <material name="red" />
+            </visual>
+        </link>
     </xacro:macro>
 </robot>

File: dogbot_hardware/description/ros2_control/dogbot.ros2_control.xacro (robot description, xacro)
@@ -11,4 +11,5 @@
                 <param name="servo_forearm_name">servo_forearm_joint</param>
                 <param name="servo_gripper_name">servo_gripper_joint</param>
+                <param name="sonar_name">sonar_joint</param>
                 <param name="device">/dev/arduino</param>
                 <param name="baud_rate">115200</param>
@@ -38,4 +39,7 @@
                 <command_interface name="position" />
             </joint>
+            <joint name="${prefix}sonar_joint">
+                <state_interface name="position" />
+            </joint>
         </ros2_control>
     </xacro:macro>
